File: Simplex/Hardware/PCB/simplex_pcb_front/simplex_pcb_front.kicad_pcb (KiCad board)
At the start: 2 copper layers, 20 x 100 mm, 17 parts, among them J1 THONKICONN, J2 THONKICONN, J3 THONKICONN, J4 THONKICONN, J5 Conn_01x07_Female, J6 Conn_01x03_Female

Commit message: updated and converted simplex to new kicad version
Other:
- net class Default removed
- net class Power removed
