File: modules/Mixer/PCBs/mixer_pcb/mixer_pcb.kicad_pcb (KiCad board)
At the start: 2 copper layers, 40 x 100 mm, 38 parts, among them J1 THONKICONN, J2 THONKICONN, J3 THONKICONN, J4 THONKICONN, J5 THONKICONN, J6 THONKICONN, J7 Eurorack_2x5_Power, J8 Conn_01x02_Socket, J9 Conn_01x02_Socket, SW1 TAIWAY 200CWMSP1T3B4M2, SW2 TAIWAY 200CWMSP1T3B4M2, SW3 TAIWAY 200CWMSP1T3B4M2, SW4 TAIWAY 200CWMSP1T3B4M2, SW5 TAIWAY 200CWMSP1T3B4M2, U1 Opamp_Dual

Commit message: move mixer to active modules
Parts:
- C3, C4: value 100pF -> 33pF
Connections:
- C3 pad 1: Net-(U1A-+) -> Net-(U1A--)
- R1 pad 2: Net-(U1A-+) -> Net-(U1A--)
- R2 pad 2: Net-(U1A-+) -> Net-(U1A--)
- R3 pad 2: Net-(U1A-+) -> Net-(U1A--)
- R4 pad 2: Net-(U1A-+) -> Net-(U1A--)
- R5 pad 2: Net-(U1A-+) -> Net-(U1A--)
- R6 pad 2: Net-(U1A-+) -> Net-(U1A--)
- R7 pad 1: Net-(U1A-+) -> Net-(U1A--)
- U1 pad 2: GND -> Net-(U1A--)
- U1 pad 3: Net-(U1A-+) -> GND
Routing:
- net Net-(U1A--): track 0.00 -> 107.4 mm
- net Net-(U1A-+): track 107.1 -> 0.00 mm
- net GND: track 308.0 -> 309.0 mm

Commit message: update mixer schematic
Parts:
- RV1, RV2, RV3, RV4: value R_Potentiometer -> A100k
Other:
- board text added: "-12v"

Commit message: update LED resistor value
Parts:
- R11: value 470Ω -> 4k7Ω
Changed lines of the file:
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@@
         (effects (font (size 1 1) (thickness 0.15)) (justify mirror))
     )
-    (fp_text value "470Ω" (at 5.08 -2.37 90) (layer "B.Fab")
+    (fp_text value "4k7Ω" (at 5.08 -2.37 90) (layer "B.Fab")
         (effects (font (size 1 1) (thickness 0.15)) (justify mirror))
     )

Commit message: adjust mixer PCB
Parts:
- moved G*** 39.1 mm to (72.4, 29.8)
- moved C5 25.7 mm to (87.6, 48.4)
- moved C6 25.6 mm to (59.7, 47.1)
- moved J7 23.3 mm to (68.6, 45.1), turned to -90 degrees
- moved J9 22.2 mm to (94.0, 120.0)
- moved R8 19.1 mm to (93.3, 69.8), turned to 180 degrees
- moved R9 17.4 mm to (93.3, 66.7)
- moved RV1 11.2 mm to (85.1, 43.1), turned to 90 degrees
- moved RV3 11.2 mm to (85.1, 83.7), turned to 90 degrees
- moved RV4 11.2 mm to (85.1, 104.0), turned to 90 degrees
- moved RV2 11.2 mm to (85.1, 63.4), turned to 90 degrees
- moved C1 8.98 mm to (76.2, 78.7)
- moved R10 5.72 mm to (94.0, 106.0)
- moved R5 4.02 mm to (68.6, 106.7)
- moved R6 4.02 mm to (68.6, 110.5)
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Routing:
- net GND: track 309.0 -> 210.9 mm
- net -12V: track 102.3 -> 60.5 mm
- net +12V: track 98.6 -> 66.9 mm
- net Net-(U1A--): track 107.4 -> 80.4 mm
- net Net-(J9-Pin_2): track 22.5 -> 7.32 mm
- net Net-(SW2-B): track 10.0 -> 24.8 mm
- net Net-(SW3-B): track 9.93 -> 23.6 mm
- net Net-(R3-Pad1): track 7.40 -> 19.3 mm
- net Net-(SW4-B): track 9.93 -> 20.9 mm
- net Net-(SW1-B): track 9.93 -> 20.8 mm
- net Net-(C3-Pad2): track 62.3 -> 70.4 mm
- net Net-(C4-Pad2): track 59.1 -> 65.7 mm
- net Net-(R1-Pad1): track 28.8 -> 23.1 mm
- net Net-(J6-Pad3): track 12.6 -> 8.12 mm
- net Net-(SW5-B): track 7.93 -> 11.7 mm
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Other:
- board text added: "+"
- board text added: "Mixer v2.1"
- board text removed: "Mixer v0.4"
