File: modules/Boost/PCBs/boost_pcb/boost_pcb.kicad_pcb (KiCad board)
At the start: 2 copper layers, 20 x 100 mm, 29 parts, among them J1 2x5 IDC, J2 THONKICONN, J3 THONKICONN, Q1 2N3904, U1 TL074

Commit message: Fix boost format
Parts:
- renumbered REF** to G1
Changed lines of the file:
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@@
 		(layer "B.Cu")
 		(at 35.56 38.1 90)
-		(property "Reference" "REF**"
+		(property "Reference" "G1"
 			(at 0 2.1 -90)
 			(unlocked yes)
