File: modules/Logic/PCBs/logic_pcb/analog.kicad_sch (KiCad schematic)
At the start: 28 parts, among them U3 LM324, U4 LM324, U5 TL072

Commit message: Switch ALU to SMD components
Parts:
- C2, C3, C4: footprint Capacitor_THT:C_Disc_D4.7mm_W2.5mm_P5.00mm -> Capacitor_SMD:C_0805_2012Metric_Pad1.18x1.45mm_HandSolder; JLC (none) -> C376974
- D1, D2, D3: footprint Diode_THT:D_DO-35_SOD27_P7.62mm_Horizontal -> Diode_SMD:D_SOD-123; JLC (none) -> C5443965
- R11, R12, R13, R15, R19, R20, R21, R22, R23, R24, R25, R26: footprint Resistor_THT:R_Axial_DIN0207_L6.3mm_D2.5mm_P10.16mm_Horizontal -> Resistor_SMD:R_0805_2012Metric_Pad1.20x1.40mm_HandSolder; JLC (none) -> C17414
- R14, R17, R18, R27, R28, R29: footprint Resistor_THT:R_Axial_DIN0207_L6.3mm_D2.5mm_P10.16mm_Horizontal -> Resistor_SMD:R_0805_2012Metric_Pad1.20x1.40mm_HandSolder; JLC (none) -> C17513
- R16: footprint Resistor_THT:R_Axial_DIN0207_L6.3mm_D2.5mm_P10.16mm_Horizontal -> Resistor_SMD:R_0805_2012Metric_Pad1.20x1.40mm_HandSolder; JLC (none) -> C57246
- U3, U4: footprint Package_DIP:DIP-14_W7.62mm -> Package_SO:SOIC-14_3.9x8.7mm_P1.27mm; JLC (none) -> C7943
- U5: footprint Package_DIP:DIP-8_W7.62mm -> Package_SO:SOP-8_3.9x4.9mm_P1.27mm; JLC (none) -> C5310783

Commit message: Get logic and quant ready for fab
Parts:
- R16: JLC C57246 -> C149504
Changed lines of the file:
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@@
 			)
 		)
-		(property "JLC" "C57246"
+		(property "JLC" "C149504"
 			(at 156.21 90.17 0)
 			(effects

Commit message: Fix wrong pin ordering on logic front; bump both boards to v1.0
Other:
- company: (none) -> Free Modular
- title: (none) -> ALU
Changed lines of the file:
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@@
 	(generator_version "9.0")
 	(paper "A4")
+	(title_block
+		(title "ALU")
+		(date "2025-04-18")
+		(rev "v1.0")
+		(company "Free Modular")
+	)
 	(junction
 		(at 95.25 46.99)
