File: modules/Quantizer/PCBs/quantizer_pcb/quantizer_pcb.kicad_sch (KiCad schematic)
At the start: 8 parts, among them J11 Conn_01x10_Socket, J12 Conn_01x08_Socket, J13 Conn_01x10_Pin, J14 Conn_01x08_Pin

Commit message: Update quant PCB to v0.2
Parts:
- J12: footprint Connector_PinSocket_2.54mm:PinSocket_1x08_P2.54mm_Vertical -> Connector_PinSocket_2.54mm:PinSocket_1x09_P2.54mm_Vertical; symbol Connector:Conn_01x08_Socket -> Connector:Conn_01x09_Socket
- J14: footprint Connector_PinSocket_2.54mm:PinSocket_1x08_P2.54mm_Vertical -> Connector_PinSocket_2.54mm:PinSocket_1x09_P2.54mm_Vertical; symbol Connector:Conn_01x08_Pin -> Connector:Conn_01x09_Pin
Connections:
- net Front Panel/btn_load: now also J12.2 (Pin_2); no longer J12.1 (Pin_1)
- net Front Panel/btn_save: now also J12.3 (Pin_3); no longer J12.2 (Pin_2)
- net Front Panel/led_input_b: now also J12.6 (Pin_6); no longer J12.5 (Pin_5)
- net Front Panel/led_output_b: now also J12.7 (Pin_7); no longer J12.6 (Pin_6)
- net Front Panel/sample_gate_b: now also J12.5 (Pin_5); no longer J12.4 (Pin_4)
- net Front Panel/trig_out_b: now also J12.8 (Pin_8); no longer J12.7 (Pin_7)
- net Front Panel/vpo_in_b: now also J12.4 (Pin_4); no longer J12.3 (Pin_3)
- net Front Panel/vpo_out_b: now also J12.9 (Pin_9); no longer J12.8 (Pin_8)
- net Rear Panel/btn_load: now also J14.2 (Pin_2); no longer J14.1 (Pin_1)
- net Rear Panel/btn_save: now also J14.3 (Pin_3); no longer J14.2 (Pin_2)
- net Rear Panel/led_input_b: now also J14.6 (Pin_6); no longer J14.5 (Pin_5)
- net Rear Panel/led_output_b: now also J14.7 (Pin_7); no longer J14.6 (Pin_6)
- net Rear Panel/sample_gate_b: now also J14.5 (Pin_5); no longer J14.4 (Pin_4)
- net Rear Panel/trig_out_b: now also J14.8 (Pin_8); no longer J14.7 (Pin_7)
- net Rear Panel/vpo_in_b: now also J14.4 (Pin_4); no longer J14.3 (Pin_3)
- net Rear Panel/vpo_out_b: now also J14.9 (Pin_9); no longer J14.8 (Pin_8)
- new net Front Panel/vref_+5: J12.1 (Pin_1)
- new net Rear Panel/vref_+5: J14.1 (Pin_1)
Other:
- sheet Front Panel ports: added vref_+5; removed none
- sheet Rear Panel ports: added vref_+5; removed none
Changed lines of the file:
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@@
 	(title_block
 		(title "Quantizer")
-		(date "2024-12-18")
-		(rev "v0.1")
+		(date "2025-04-02")
+		(rev "v0.2")
 		(company "Free Modular")
 	)
@@
 	(wire
 		(pts
+			(xy 99.06 106.68) (xy 107.95 106.68)
+		)
+		(stroke
+			(width 0)
+			(type default)
+		)
+	)
+	(wire
+		(pts
 			(xy 120.65 60.96) (xy 129.54 60.96)
 		)
@@
 		(pts
 			(xy 120.65 76.2) (xy 129.54 76.2)
+		)
+		(stroke
+			(width 0)
+			(type default)
+		)
+	)
+	(wire
+		(pts
+			(xy 120.65 106.68) (xy 129.54 106.68)
 		)
 		(stroke
@@
 	)
 	(symbol
-		(lib_id "Connector:Conn_01x08_Pin")
-		(at 115.57 93.98 0)
+		(lib_id "Connector:Conn_01x09_Pin")
+		(at 115.57 96.52 0)
 		(unit 1)
 		(exclude_from_sim no)
@@
 		(dnp no)
 		(property "Reference" "J14"
-			(at 117.348 107.95 90)
+			(at 117.348 110.49 90)
 			(effects
 				(font
@@
 		)
 		(property "Value" "Conn_01x08_Pin"
-			(at 119.634 114.046 90)
-			(effects
-				(font
-					(size 1.27 1.27)
-				)
-			)
-		)
-		(property "Footprint" "Connector_PinSocket_2.54mm:PinSocket_1x08_P2.54mm_Vertical"
-			(at 115.57 93.98 0)
+			(at 119.634 116.586 90)
+			(effects
+				(font
+					(size 1.27 1.27)
+				)
+			)
+		)
+		(property "Footprint" "Connector_PinSocket_2.54mm:PinSocket_1x09_P2.54mm_Vertical"
+			(at 115.57 96.52 0)
 			(effects
 				(font
@@
 		)
 		(property "Datasheet" "~"
-			(at 115.57 93.98 0)
-			(effects
-				(font
-					(size 1.27 1.27)
-				)
-				(hide yes)
-			)
-		)
-		(property "Description" "Generic connector, single row, 01x08, script generated"
-			(at 115.57 93.98 0)
+			(at 115.57 96.52 0)
+			(effects
+				(font
+					(size 1.27 1.27)
+				)
+				(hide yes)
+			)
+		)
+		(property "Description" "Generic connector, single row, 01x09, script generated"
+			(at 115.57 96.52 0)
 			(effects
 				(font
@@
 		)
 		(pin "6"
+		)
+		(pin "9"
 		)
 		(instances
@@
 	)
 	(symbol
-		(lib_id "Connector:Conn_01x08_Socket")
-		(at 113.03 93.98 0)
+		(lib_id "Connector:Conn_01x09_Socket")
+		(at 113.03 96.52 0)
 		(unit 1)
 		(exclude_from_sim no)
@@
 		(dnp no)
 		(property "Reference" "J12"
-			(at 109.22 109.474 90)
+			(at 109.22 112.014 90)
 			(effects
 				(font
@@
 		)
 		(property "Value" "Conn_01x08_Socket"
-			(at 111.76 124.968 90)
-			(effects
-				(font
-					(size 1.27 1.27)
-				)
-				(justify left)
-			)
-		)
-		(property "Footprint" "Connector_PinSocket_2.54mm:PinSocket_1x08_P2.54mm_Vertical"
-			(at 113.03 93.98 0)
+			(at 111.76 127.508 90)
+			(effects
+				(font
+					(size 1.27 1.27)
+				)
+				(justify left)
+			)
+		)
+		(property "Footprint" "Connector_PinSocket_2.54mm:PinSocket_1x09_P2.54mm_Vertical"
+			(at 113.03 96.52 0)
 			(effects
 				(font
@@
 		)
 		(property "Datasheet" "~"
-			(at 113.03 93.98 0)
-			(effects
-				(font
-					(size 1.27 1.27)
-				)
-				(hide yes)
-			)
-		)
-		(property "Description" "Generic connector, single row, 01x08, script generated"
-			(at 113.03 93.98 0)
+			(at 113.03 96.52 0)
+			(effects
+				(font
+					(size 1.27 1.27)
+				)
+				(hide yes)
+			)
+		)
+		(property "Description" "Generic connector, single row, 01x09, script generated"
+			(at 113.03 96.52 0)
 			(effects
 				(font
@@
 		)
 		(pin "8"
+		)
+		(pin "9"
 		)
 		(instances
@@
 		)
 		(pin "trig_out_b" output
+			(at 99.06 104.14 0)
+			(effects
+				(font
+					(size 1.27 1.27)
+				)
+				(justify right)
+			)
+		)
+		(pin "vpo_out_b" output
+			(at 99.06 106.68 0)
+			(effects
+				(font
+					(size 1.27 1.27)
+				)
+				(justify right)
+			)
+		)
+		(pin "vpo_in_b" output
+			(at 99.06 93.98 0)
+			(effects
+				(font
+					(size 1.27 1.27)
+				)
+				(justify right)
+			)
+		)
+		(pin "sample_gate_b" output
+			(at 99.06 96.52 0)
+			(effects
+				(font
+					(size 1.27 1.27)
+				)
+				(justify right)
+			)
+		)
+		(pin "led_input_b" input
+			(at 99.06 99.06 0)
+			(effects
+				(font
+					(size 1.27 1.27)
+				)
+				(justify right)
+			)
+		)
+		(pin "led_output_b" input
 			(at 99.06 101.6 0)
-			(effects
-				(font
-					(size 1.27 1.27)
-				)
-				(justify right)
-			)
-		)
-		(pin "vpo_out_b" output
-			(at 99.06 104.14 0)
-			(effects
-				(font
-					(size 1.27 1.27)
-				)
-				(justify right)
-			)
-		)
-		(pin "vpo_in_b" output
-			(at 99.06 91.44 0)
-			(effects
-				(font
-					(size 1.27 1.27)
-				)
-				(justify right)
-			)
-		)
-		(pin "sample_gate_b" output
-			(at 99.06 93.98 0)
-			(effects
-				(font
-					(size 1.27 1.27)
-				)
-				(justify right)
-			)
-		)
-		(pin "led_input_b" input
-			(at 99.06 96.52 0)
-			(effects
-				(font
-					(size 1.27 1.27)
-				)
-				(justify right)
-			)
-		)
-		(pin "led_output_b" input
-			(at 99.06 99.06 0)
 			(effects
 				(font
@@
 		)
 		(pin "btn_save" output
-			(at 99.06 88.9 0)
+			(at 99.06 91.44 0)
 			(effects
 				(font
@@
 		)
 		(pin "btn_load" output
-			(at 99.06 86.36 0)
+			(at 99.06 88.9 0)
 			(effects
 				(font
@@
 		(pin "resistor_ladder_voltage" output
 			(at 99.06 66.04 0)
+			(effects
+				(font
+					(size 1.27 1.27)
+				)
+				(justify right)
+			)
+		)
+		(pin "vref_+5" input
+			(at 99.06 86.36 0)
 			(effects
 				(font
@@
 		)
 		(pin "btn_load" input
-			(at 129.54 86.36 180)
+			(at 129.54 88.9 180)
 			(effects
 				(font
@@
 		)
 		(pin "btn_save" input
-			(at 129.54 88.9 180)
+			(at 129.54 91.44 180)
 			(effects
 				(font
@@
 		)
 		(pin "vpo_out_b" output
-			(at 129.54 104.14 180)
+			(at 129.54 106.68 180)
 			(effects
 				(font
@@
 		)
 		(pin "vpo_in_b" input
-			(at 129.54 91.44 180)
+			(at 129.54 93.98 180)
 			(effects
 				(font
@@
 		)
 		(pin "sample_gate_b" input
-			(at 129.54 93.98 180)
+			(at 129.54 96.52 180)
 			(effects
 				(font
@@
 		)
 		(pin "led_output_b" output
+			(at 129.54 101.6 180)
+			(effects
+				(font
+					(size 1.27 1.27)
+				)
+				(justify left)
+			)
+		)
+		(pin "led_input_b" output
 			(at 129.54 99.06 180)
-			(effects
-				(font
-					(size 1.27 1.27)
-				)
-				(justify left)
-			)
-		)
-		(pin "led_input_b" output
-			(at 129.54 96.52 180)
 			(effects
 				(font
@@
 		)
 		(pin "trig_out_b" output
-			(at 129.54 101.6 180)
-			(effects
-				(font
+			(at 129.54 104.14 180)
+			(effects
+				(font
+					(size 1.27 1.27)
+				)
+				(justify left)
+			)
+		)
+		(pin "vref_+5" output
+			(at 129.54 86.36 180)
+			(effects
+				(font

Commit message: Working on quantizer documentation
Parts:
- J12: value Conn_01x08_Socket -> Conn_01x09_Socket
- J14: value Conn_01x08_Pin -> Conn_01x09_Pin
Changed lines of the file:
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@@
 			)
 		)
-		(property "Value" "Conn_01x08_Pin"
+		(property "Value" "Conn_01x09_Pin"
 			(at 119.634 116.586 90)
 			(effects
@@
 			)
 		)
-		(property "Value" "Conn_01x08_Socket"
+		(property "Value" "Conn_01x09_Socket"
 			(at 111.76 127.508 90)
 			(effects
