File: modules/Lights/PCBs/lights_pcb/front_board.kicad_sch (KiCad schematic)
At the start: 6 parts, among them J1 THONKICONN, J2 THONKICONN, J3 THONKICONN, J4 THONKICONN, SW1 TL1105SPF250Q

Commit message: Knobcon demo
Other:
- company: (none) -> Free Modular
- title: (none) -> Lights
Changed lines of the file:
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@@
 	(generator_version "9.0")
 	(paper "A4")
+	(title_block
+		(title "Lights")
+		(date "2025-08-27")
+		(rev "v0.2")
+		(company "Free Modular")
+	)
 	(junction
 		(at 63.5 111.76)

Commit message: Lights 0.2 revision
Changed lines of the file:
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@@
 	(title_block
 		(title "Lights")
-		(date "2025-08-27")
+		(date "2025-10-13")
 		(rev "v0.2")
 		(company "Free Modular")
@@
 	(wire
 		(pts
+			(xy 95.25 71.12) (xy 101.6 71.12)
+		)
+		(stroke
+			(width 0)
+			(type default)
+		)
+	)
+	(wire
+		(pts
 			(xy 73.66 63.5) (xy 73.66 60.96)
 		)
@@
 	(wire
 		(pts
-			(xy 99.06 73.66) (xy 99.06 71.12)
+			(xy 95.25 73.66) (xy 95.25 71.12)
 		)
 		(stroke
@@
 	(wire
 		(pts
-			(xy 99.06 71.12) (xy 101.6 71.12)
-		)
-		(stroke
-			(width 0)
-			(type default)
-		)
-	)
-	(wire
-		(pts
 			(xy 73.66 111.76) (xy 73.66 109.22)
 		)
@@
 	(hierarchical_label "GND"
 		(shape input)
-		(at 99.06 73.66 270)
+		(at 95.25 73.66 270)
 		(effects
 			(font
@@
 		)
 	)
+	(netclass_flag ""
+		(length 2.54)
+		(shape round)
+		(at 95.25 71.12 0)
+		(fields_autoplaced yes)
+		(effects
+			(font
+				(size 1.27 1.27)
+			)
+			(justify left bottom)
+		)
+		(property "Netclass" "Power"
+			(at 95.9485 68.58 0)
+			(effects
+				(font
+					(size 1.27 1.27)
+				)
+				(justify left)
+			)
+		)
+		(property "Component Class" ""
+			(at -43.18 -64.77 0)
+			(effects
+				(font
+					(size 1.27 1.27)
+					(italic yes)
+				)
+			)
+		)
+	)
