File: modules/Lights/PCBs/lights_pcb/led_driver.kicad_sch (KiCad schematic)
At the start: 18 parts, among them J5 Conn_01x04_Pin, J6 Conn_01x03_Pin, J8 Barrel_Jack, Q1 2N7000, Q2 IRF9510PBF, Q3 2N7000, Q4 IRF9510PBF, Q5 2N7000, Q6 IRF9510PBF, U3 ISO6740, U4 LM4040BIZ-5

Commit message: Knobcon demo
Parts:
- removed Q2, Q4, Q6: IRF9510PBF, Package_TO_SOT_THT:TO-220-3_Vertical, symbol Transistor_FET:IRF9540N
- removed Q5: 2N7000, Package_TO_SOT_THT:TO-92_Inline, symbol Transistor_FET:2N7000
- removed R14, R15: 2.2kΩ, Resistor_THT:R_Axial_DIN0207_L6.3mm_D2.5mm_P7.62mm_Horizontal, symbol Device:R
- added Q2: RFP30N06LE, Package_TO_SOT_THT:TO-220-3_Vertical, symbol Transistor_FET:2N7000
- added Q7, Q8: 2N7000, Package_TO_SOT_THT:TO-92_Inline, symbol Transistor_FET:2N7000
- added R19, R20: 1kΩ, Resistor_THT:R_Axial_DIN0207_L6.3mm_D2.5mm_P7.62mm_Horizontal, symbol Device:R
- Q1, Q3: value 2N7000 -> RFP30N06LE; footprint Package_TO_SOT_THT:TO-92_Inline -> Package_TO_SOT_THT:TO-220-3_Vertical
- R13: value 2.2kΩ -> 100Ω
- R16: value 6.2kΩ -> 470Ω
Connections:
- net LED_ANODE_B: now also Q3.2 (D)
- net LED_ANODE_G: now also Q2.2 (D)
- net LED_GND: now also Q2.1 (S), Q7.1 (S), Q8.1 (S)
- net LED_PWR: now also R19.2, R20.2; no longer R13.1
- net at Q1.3 (G): now also U3.14 (OUTA); no longer R13.2
- net at Q3.3 (G): now also U3.12 (OUTC)
- net LED_CATHODE_R: now reaches Q1.2 (D)
- net LED_CATHODE_R: no longer U3.14 (OUTA)
- net at R18.1: now also Q8.3 (D), R20.1; no longer U3.11 (OUTD)
- net at U3.13 (OUTB): now also Q2.3 (G); no longer Q3.2 (G)
- new net: R13.2, U3.11 (OUTD)
- new net: Q7.3 (D), Q8.2 (G), R19.1
- new net: Q7.2 (G), R13.1
Other:
- company: (none) -> Free Modular
- title: (none) -> Lights
- moved on the sheet: C5, Q1, R16, R18, U4

Commit message: Lights 0.2 revision
Parts:
- added SW2: SW_SPDT, Button_Switch_THT:SW_Slide-03_Wuerth-WS-SLTV_10x2.5x6.4_P2.54mm, symbol Switch:SW_SPDT_312
- renumbered R16 to R21
Connections:
- net LED_CATHODE_R is gone; now on net LED_ANODE_R: Q1.2 (D)
- net LED_5V: now also SW2.1 (B); no longer C5.1, R21.2, U4.2 (K)
- net LED_GND: no longer J5.1 (Pin_1)
- net LED_PWR: now also J5.1 (Pin_1), SW2.2 (C)
- new net: C5.1, R21.2, SW2.3 (A), U4.2 (K)
Other:
- moved on the sheet: C5
