File: modules/Lights/PCBs/lights_pcb/lights_pcb.kicad_pcb (KiCad board)
At the start: 2 copper layers, 89 x 100 mm, 51 parts, among them J1 THONKICONN, J10 Conn_02x04_Top_Bottom, J11 Conn_02x04_Top_Bottom, J12 Conn_02x02_Top_Bottom, J13 Conn_02x02_Top_Bottom, J2 THONKICONN, J3 THONKICONN, J4 THONKICONN, J5 Conn_01x04_Pin, J6 Conn_01x03_Pin, J8 Barrel_Jack, J9 Eurorack_2x8_Power, Q1 2N7000, Q2 IRF9510PBF, Q3 2N7000, Q4 IRF9510PBF, Q5 2N7000, Q6 IRF9510PBF, SW1 TL1105SPF250Q, U1 MCP6004, U2 CD4051B, U3 ISO6740, U4 LM4040BIZ-5, U5 LM4040BIZ-5

Commit message: v0.1 biodata pcb
Parts:
- added REF**: logo_small, FreeModular:logo_small, B.Cu at (134.0, 43.5)
Other:
- board text added: "Free Modular Lights back v0.1"
- board text added: "Free Modular Lights front v0.1"
- board text added: "this machine kills fascists"
- board text added: "this side towards center of module"
- board text removed: "Lights back v0.1"
- board text removed: "Lights front v0.1"

Commit message: Ready for build and export
Parts:
- added B1: Board, kikit:Board, F.Cu at (63.5, 31.8)
- added B2: Board, kikit:Board, F.Cu at (120.2, 31.8)
Other:
- board text added: "perpendicular PCB goes here"
Changed lines of the file:
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@@
 		)
 	)
+	(footprint "kikit:Board"
+		(layer "F.Cu")
+		(at 63.5 31.75)
+		(descr "Mark board for extraction")
+		(property "Reference" "B1"
+			(at -4.5 -5 0)
+			(layer "Dwgs.User")
+			(effects
+				(font
+					(size 1 1)
+					(thickness 0.15)
+				)
+				(justify left)
+			)
+		)
+		(property "Value" "Board"
+			(at -7.25 -5 0)
+			(layer "Dwgs.User")
+			(effects
+				(font
+					(size 1 1)
+					(thickness 0.15)
+				)
+			)
+		)
+		(property "Datasheet" ""
+			(at 0 0 0)
+			(unlocked yes)
+			(layer "F.Fab")
+			(hide yes)
+			(effects
+				(font
+					(size 1.27 1.27)
+					(thickness 0.15)
+				)
+			)
+		)
+		(property "Description" ""
+			(at 0 0 0)
+			(unlocked yes)
+			(layer "F.Fab")
+			(hide yes)
+			(effects
+				(font
+					(size 1.27 1.27)
+					(thickness 0.15)
+				)
+			)
+		)
+		(attr through_hole)
+		(fp_line
+			(start -1.25 -4)
+			(end -9.25 -4)
+			(stroke
+				(width 0.2)
+				(type solid)
+			)
+			(layer "Dwgs.User")
+		)
+		(fp_line
+			(start 0 0)
+			(end -1.25 -4)
+			(stroke
+				(width 0.2)
+				(type solid)
+			)
+			(layer "Dwgs.User")
+		)
+		(fp_line
+			(start 0 0)
+			(end -1 -0.5)
+			(stroke
+				(width 0.2)
+				(type solid)
+			)
+			(layer "Dwgs.User")
+		)
+		(fp_line
+			(start 0 0)
+			(end 0.5 -1)
+			(stroke
+				(width 0.2)
+				(type solid)
+			)
+			(layer "Dwgs.User")
+		)
+		(embedded_fonts no)
+	)
 	(footprint "Connector_PinSocket_2.54mm:PinSocket_1x03_P2.54mm_Vertical"
 		(layer "F.Cu")
@@
 		)
 	)
+	(footprint "kikit:Board"
+		(layer "F.Cu")
+		(at 120.25 31.75)
+		(descr "Mark board for extraction")
+		(property "Reference" "B2"
+			(at -4.5 -5 0)
+			(layer "Dwgs.User")
+			(effects
+				(font
+					(size 1 1)
+					(thickness 0.15)
+				)
+				(justify left)
+			)
+		)
+		(property "Value" "Board"
+			(at -7.25 -5 0)
+			(layer "Dwgs.User")
+			(effects
+				(font
+					(size 1 1)
+					(thickness 0.15)
+				)
+			)
+		)
+		(property "Datasheet" ""
+			(at 0 0 0)
+			(unlocked yes)
+			(layer "F.Fab")
+			(hide yes)
+			(effects
+				(font
+					(size 1.27 1.27)
+					(thickness 0.15)
+				)
+			)
+		)
+		(property "Description" ""
+			(at 0 0 0)
+			(unlocked yes)
+			(layer "F.Fab")
+			(hide yes)
+			(effects
+				(font
+					(size 1.27 1.27)
+					(thickness 0.15)
+				)
+			)
+		)
+		(attr through_hole)
+		(fp_line
+			(start -1.25 -4)
+			(end -9.25 -4)
+			(stroke
+				(width 0.2)
+				(type solid)
+			)
+			(layer "Dwgs.User")
+		)
+		(fp_line
+			(start 0 0)
+			(end -1.25 -4)
+			(stroke
+				(width 0.2)
+				(type solid)
+			)
+			(layer "Dwgs.User")
+		)
+		(fp_line
+			(start 0 0)
+			(end -1 -0.5)
+			(stroke
+				(width 0.2)
+				(type solid)
+			)
+			(layer "Dwgs.User")
+		)
+		(fp_line
+			(start 0 0)
+			(end 0.5 -1)
+			(stroke
+				(width 0.2)
+				(type solid)
+			)
+			(layer "Dwgs.User")
+		)
+		(embedded_fonts no)
+	)
 	(footprint "FreeModular:THONKICONN"
 		(layer "F.Cu")
@@
 	)
 	(gr_line
+		(start 59.69 73.66)
+		(end 59.69 52.705)
+		(stroke
+			(width 0.3)
+			(type solid)
+		)
+		(layer "B.SilkS")
+	)
+	(gr_line
+		(start 59.69 113.665)
+		(end 59.69 92.71)
+		(stroke
+			(width 0.3)
+			(type solid)
+		)
+		(layer "B.SilkS")
+	)
+	(gr_line
 		(start 120.25 31.75)
 		(end 147.75 31.75)
@@
 		)
 	)
+	(gr_text "perpendicular PCB goes here"
+		(at 59.69 83.185 90)
+		(layer "B.SilkS")
+		(effects
+			(font
+				(size 0.8 0.8)
+				(thickness 0.1)
+			)
+			(justify mirror)
+		)
+	)

Commit message: Knobcon demo
Parts:
- removed B1, B2: Board, kikit:Board
- removed Q4, Q6: IRF9510PBF, Package_TO_SOT_THT:TO-220-3_Vertical
- removed Q5: 2N7000, Package_TO_SOT_THT:TO-92_Inline
- removed R14, R15: 2.2kΩ, Resistor_THT:R_Axial_DIN0207_L6.3mm_D2.5mm_P7.62mm_Horizontal
- removed REF**: logo_small, FreeModular:logo_small
- added Q7: 2N7000, Package_TO_SOT_THT:TO-92_Inline, F.Cu at (174.0, 122.5)
- added Q8: 2N7000, Package_TO_SOT_THT:TO-92_Inline, F.Cu at (174.0, 128.3)
- added R19: 1kΩ, Resistor_THT:R_Axial_DIN0207_L6.3mm_D2.5mm_P7.62mm_Horizontal, F.Cu at (164.5, 99.5)
- added R20: 1kΩ, Resistor_THT:R_Axial_DIN0207_L6.3mm_D2.5mm_P7.62mm_Horizontal, F.Cu at (177.2, 111.1)
- Q1, Q3: value 2N7000 -> RFP30N06LE; footprint Package_TO_SOT_THT:TO-92_Inline -> Package_TO_SOT_THT:TO-220-3_Vertical
- Q2: value IRF9510PBF -> RFP30N06LE
- R1, R3, R5: value 10kΩ -> 51kΩ
- R10, R2, R4, R6: value 10kΩ -> 33kΩ
- R11, R12, R7, R8, R9: value 20kΩ -> 100kΩ
- R13: value 2.2kΩ -> 100Ω
- R16: value 6.2kΩ -> 470Ω
- moved R13 57.1 mm to (175.6, 103.8)
- moved Q2 46.8 mm to (168.6, 86.8)
- moved Q3 45.7 mm to (168.6, 92.7)
- moved Q1 36.6 mm to (160.0, 109.2)
- moved C4 13.0 mm to (107.6, 73.7), turned to 90 degrees
Connections:
- A1 pad 36: unconnected-(A1-3V3-Pad36) -> /Rear Board/+3.3V
- C4 pad 1: /Rear Board/+5V -> /Rear Board/+3.3V
- Q1 pad 2: Net-(Q1-G) -> /Rear Board/LED Driver/LED_CATHODE_R
- Q1 pad 3: Net-(Q1-D) -> Net-(Q1-G)
- Q2 pad 1: Net-(Q1-D) -> /Rear Board/LED Driver/LED_GND
- Q2 pad 2: /Rear Board/LED Driver/LED_ANODE_R -> /Rear Board/LED Driver/LED_ANODE_G
- Q2 pad 3: /Rear Board/LED Driver/LED_PWR -> Net-(Q2-G)
- Q3 pad 2: Net-(Q3-G) -> /Rear Board/LED Driver/LED_ANODE_B
- Q3 pad 3: Net-(Q3-D) -> Net-(Q3-G)
- R13 pad 1: /Rear Board/LED Driver/LED_PWR -> Net-(Q7-G)
- R13 pad 2: Net-(Q1-D) -> Net-(U3-OUTD)
- R18 pad 1: Net-(U3-OUTD) -> Net-(Q8-D)
- U1 pad 11: /Rear Board/+5V -> GND
- U1 pad 4: GND -> /Rear Board/+3.3V
- U3 pad 12: Net-(Q5-G) -> Net-(Q3-G)
- U3 pad 13: Net-(Q3-G) -> Net-(Q2-G)
Routing:
- net /Rear Board/+3.3V: track 0.00 -> 58.0 mm
- net Net-(U2-X1): track 2.53 -> 45.7 mm
- net Net-(Q5-G): track 23.6 -> 0.00 mm, vias 1 -> 0
- net Net-(Q2-G): track 0.00 -> 20.9 mm, vias 0 -> 1
- net (no net): track 0.00 -> 18.4 mm
- net Net-(U3-OUTD): track 10.4 -> 0.00 mm, vias 1 -> 0
- net Net-(Q8-D): track 0.00 -> 10.4 mm, vias 0 -> 1
- net Net-(Q5-D): track 9.57 -> 0.00 mm
- net Net-(Q3-D): track 8.78 -> 0.00 mm
- net Net-(Q1-D): track 8.78 -> 0.00 mm
- net /Rear Board/LED Driver/LED_CATHODE_R: track 0.00 -> 8.78 mm
- net /Rear Board/+5V: track 111.2 -> 114.7 mm
- net Net-(Q3-G): track 20.9 -> 23.6 mm
- net /Rear Board/LED_B: track 87.1 -> 88.4 mm
- net /Rear Board/LED_G: track 84.3 -> 85.4 mm
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Other:
- board text added: "Free Modular Lights back v0.2"
- board text removed: "Free Modular Lights back v0.1"

Commit message: Lights 0.2 revision
Parts:
- added B1: Board, kikit:Board, F.Cu at (61.1, 31.8)
- added B2: Board, kikit:Board, F.Cu at (124.5, 31.8)
- added G1: logo_small, FreeModular:logo_small, F.Cu at (134.9, 95.9)
- added R14: 470Ω, Resistor_THT:R_Axial_DIN0207_L6.3mm_D2.5mm_P7.62mm_Horizontal, F.Cu at (105.1, 56.8)
- added R15: 470Ω, Resistor_THT:R_Axial_DIN0207_L6.3mm_D2.5mm_P7.62mm_Horizontal, F.Cu at (105.1, 60.0)
- added R16: 470Ω, Resistor_THT:R_Axial_DIN0207_L6.3mm_D2.5mm_P7.62mm_Horizontal, F.Cu at (105.1, 62.9)
- added SW2: SW_SPDT, Button_Switch_THT:SW_Slide-03_Wuerth-WS-SLTV_10x2.5x6.4_P2.54mm, F.Cu at (122.6, 127.6)
- U2: value CD4051B -> SN74LVC1G3157DCKR; footprint Package_DIP:DIP-16_W7.62mm -> Package_TO_SOT_SMD:SOT-363_SC-70-6_Handsoldering
- moved R20 58.0 mm to (119.7, 119.1), turned to 180 degrees
- moved R13 56.6 mm to (119.7, 112.7), turned to 180 degrees
- moved Q3 55.0 mm to (114.3, 101.6), turned to -90 degrees
- moved Q8 52.1 mm to (122.9, 118.4), turned to -90 degrees
- moved Q7 52.0 mm to (122.9, 112.7), turned to -90 degrees
- moved R19 47.7 mm to (119.7, 115.9), turned to 180 degrees
- moved Q2 37.7 mm to (134.0, 101.6), turned to -90 degrees
- moved Q1 36.4 mm to (124.5, 101.6), turned to -90 degrees
- moved C5 31.8 mm to (107.0, 129.5)
- moved C2 13.3 mm to (134.6, 87.3), turned to 180 degrees
- moved R18 11.0 mm to (127.0, 115.6)
- moved U2 11.0 mm to (134.6, 90.5), turned to 0 degrees
- moved U4 10.5 mm to (107.4, 125.1), turned to 90 degrees
- moved U5 10.5 mm to (107.0, 53.0), turned to 0 degrees
- moved R21 9.74 mm to (119.7, 122.2), turned to 180 degrees
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- renumbered R2 to R1, R8 to R10, R9 to R11, R4 to R2, R16 to R21, R6 to R3, R10 to R4, R1 to R5, R3 to R6, R5 to R7, R11 to R8, R7 to R9
Connections:
- A1 pad 13: GND -> /Rear Board/GND
- A1 pad 18: GND -> /Rear Board/GND
- A1 pad 23: GND -> /Rear Board/GND
- A1 pad 28: GND -> /Rear Board/GND
- A1 pad 3: GND -> /Rear Board/GND
- A1 pad 32: /Rear Board/CV_MUXED -> /Rear Board/G_CV_MUXED
- A1 pad 34: unconnected-(A1-GPIO28_ADC2-Pad34) -> /Rear Board/RB_CV_MUXED
- A1 pad 38: GND -> /Rear Board/GND
- A1 pad 4: /Rear Board/LED_R -> Net-(A1-GPIO2)
- A1 pad 5: /Rear Board/LED_G -> Net-(A1-GPIO3)
- A1 pad 6: /Rear Board/LED_B -> Net-(A1-GPIO4)
- A1 pad 8: GND -> /Rear Board/GND
- A1 pad 9: Net-(A1-GPIO6) -> unconnected-(A1-GPIO6-Pad9)_1
- C1 pad 2: GND -> /Rear Board/GND
- C2 pad 1: /Rear Board/+12V -> /Rear Board/+3.3V
- C2 pad 2: GND -> /Rear Board/GND
- C3 pad 2: GND -> /Rear Board/GND
- C4 pad 2: GND -> /Rear Board/GND
- C5 pad 1: /Rear Board/LED Driver/LED_5V -> Net-(SW2-A)
- C6 pad 2: GND -> /Rear Board/GND
- J12 pad 1: GND -> /Rear Board/GND
- J12 pad 2: GND -> /Rear Board/GND
- J12 pad 3: GND -> /Rear Board/GND
- J12 pad 4: GND -> /Rear Board/GND
- J5 pad 1: /Rear Board/LED Driver/LED_GND -> /Rear Board/LED Driver/LED_PWR
- J9 pad 3: GND -> /Rear Board/GND
- J9 pad 4: GND -> /Rear Board/GND
- J9 pad 5: GND -> /Rear Board/GND
- J9 pad 6: GND -> /Rear Board/GND
- J9 pad 7: GND -> /Rear Board/GND
- J9 pad 8: GND -> /Rear Board/GND
- Q1 pad 2: /Rear Board/LED Driver/LED_CATHODE_R -> /Rear Board/LED Driver/LED_ANODE_R
- R1 pad 2: Net-(U2-X0) -> Net-(U2-B2)
- R2 pad 2: Net-(U2-X1) -> /Rear Board/G_CV_MUXED
- R21 pad 2: /Rear Board/LED Driver/LED_5V -> Net-(SW2-A)
- R3 pad 2: Net-(U2-X2) -> Net-(U2-B1)
- U1 pad 10: GND -> /Rear Board/GND
- U1 pad 11: GND -> /Rear Board/GND
- U1 pad 12: GND -> /Rear Board/GND
- U1 pad 14: Net-(U2-X2) -> Net-(U2-B1)
- U1 pad 3: GND -> /Rear Board/GND
- U1 pad 5: GND -> /Rear Board/GND
- U1 pad 7: Net-(U2-X0) -> Net-(U2-B2)
- U1 pad 8: Net-(U2-X1) -> /Rear Board/G_CV_MUXED
- U2 pad 1: unconnected-(U2-X4-Pad1) -> Net-(U2-B2)
- U2 pad 2: unconnected-(U2-X6-Pad2) -> /Rear Board/GND
- U2 pad 3: /Rear Board/CV_MUXED -> Net-(U2-B1)
- U2 pad 4: unconnected-(U2-X7-Pad4) -> /Rear Board/RB_CV_MUXED
- U2 pad 5: unconnected-(U2-X5-Pad5) -> /Rear Board/+3.3V
- U2 pad 6: GND -> Net-(A1-GPIO7)
- U3 pad 2: GND -> /Rear Board/GND
- U3 pad 8: GND -> /Rear Board/GND
- U4 pad 2: /Rear Board/LED Driver/LED_5V -> Net-(SW2-A)
- U5 pad 2: GND -> /Rear Board/GND
Routing:
- net GND: track 260.8 -> 0.00 mm
- net /Rear Board/GND: track 0.00 -> 206.4 mm
- net /Rear Board/+12V: track 132.8 -> 2.54 mm
- net /Rear Board/LED Driver/LED_PWR: track 75.7 -> 0.00 mm
- net /Rear Board/G_CV_MUXED: track 0.00 -> 62.0 mm, vias 0 -> 3
- net /Rear Board/+3.3V: track 58.0 -> 119.6 mm
- net /Rear Board/CV_MUXED: track 51.8 -> 0.00 mm
- net Net-(U2-B2): track 0.00 -> 48.8 mm, vias 0 -> 1
- net Net-(U2-X0): track 46.7 -> 0.00 mm
- net /Rear Board/RB_CV_MUXED: track 0.00 -> 46.5 mm, vias 0 -> 1
- net Net-(U2-X1): track 45.7 -> 0.00 mm
- net Net-(A1-GPIO6): track 43.1 -> 0.00 mm
- net /Rear Board/LED_B: track 88.4 -> 57.2 mm
- net /Rear Board/LED Driver/LED_5V: track 24.4 -> 51.5 mm
- net Net-(A1-GPIO4): track 0.00 -> 26.2 mm
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- added copper zone on B.Cu, net /Front Board/GND
- added copper zone on B.Cu, net /Rear Board/GND
- added copper zone on F.Cu, net /Rear Board/GND
- removed copper zone on B.Cu, net GND
- removed copper zone on F.Cu, net GND
Other:
- outline, holes or cut-outs redrawn
- board text added: "5V"
- board text added: "9-12V"
- board text removed: "K"
