File: modules/Lights/PCBs/lights_pcb/lights_pcb.kicad_sch (KiCad schematic)
At the start: 4 parts, among them J10 Conn_02x04_Top_Bottom, J11 Conn_02x04_Top_Bottom, J12 Conn_02x02_Top_Bottom, J13 Conn_02x02_Top_Bottom

Commit message: Knobcon demo
Other:
- company: (none) -> Free Modular
- title: (none) -> Lights
Changed lines of the file:
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@@
 	(generator_version "9.0")
 	(paper "A4")
+	(title_block
+		(title "Lights")
+		(date "2025-08-27")
+		(rev "v0.2")
+		(company "Free Modular")
+	)
 	(junction
 		(at 146.05 86.36)
